Commit message: Bot made into front wheel drive and controls plugin errors resolved

File: simulation/eklavya5_description/robots/chasisss.urdf.xacro (robot description, xacro)
@@ -3,15 +3,11 @@
   name="chasisss"
   xmlns:sensor="http://playerstage.sourceforge.net/gazebo/xmlschema/#sensor"
-  xmlns:controller="http://playerstage.sourceforge.net/gazebo/xmlschema/#controller"
-  xmlns:interface="http://playerstage.sourceforge.net/gazebo/xmlschema/#interface"
-  xmlns:xacro="http://ros.org/wiki/xacro">
-  <!-- Included URDF/XACRO Files -->
-  <xacro:include filename="$(find eklavya5_description)/sensors/camera.urdf.xacro" />
-  <xacro:include filename="$(find eklavya5_description)/sensors/lidar.urdf.xacro" />
-  <xacro:include filename="$(find eklavya5_description)/sensors/imu.urdf.xacro" />
-  <xacro:include filename="$(find eklavya5_description)/sensors/gps.urdf.xacro" />
-  <!-- PROPERTY LIST -->
-  <property name="M_PI" value="3.1415926535897931" />
-  <!--PARTS-->
+xmlns:controller="http://playerstage.sourceforge.net/gazebo/xmlschema/#controller"
+xmlns:interface="http://playerstage.sourceforge.net/gazebo/xmlschema/#interface"
+xmlns:xacro="http://ros.org/wiki/xacro"
+>
+<xacro:include filename="$(find eklavya5_description)/sensors/imu.urdf.xacro" />
+<xacro:include filename="$(find eklavya5_description)/sensors/gps.urdf.xacro" />
+ <property name="M_PI" value="3.1415926535897931" />
   <link
     name = "base_link">
@@ -24,12 +20,12 @@
         rpy="0 0 0" />
       <mass
-        value="1.3372" />
+        value="1.60779" />
       <inertia
-        ixx="0.11623"
-        ixy="-0.003745"
-        ixz="-0.038661"
-        iyy="0.10504"
-        iyz="-0.010842"
-        izz="0.086997" />
+        ixx="0.100657"
+        ixy="0.000429"
+        ixz="-0.012951"
+        iyy="0.062637"
+        iyz="-0.000032"
+        izz="0.126211" />
     </inertial>
     <visual>
@@ -75,12 +71,12 @@
         rpy="0 0 0" />
       <mass
-        value="0.50841" />
+        value="5.15679" />
       <inertia
-        ixx="0.012612"
-        ixy="-8.93E-06"
-        ixz="-0.00091193"
-        iyy="0.0089584"
-        iyz="0.00011487"
-        izz="0.0042882" />
+        ixx="0.030405"
+        ixy="0.00"
+        ixz="-0.014212"
+        iyy="0.037062"
+        iyz="0.00"
+        izz="0.015136" />
     </inertial>
     <visual>
@@ -111,8 +107,8 @@
     name="Chassis-Steering"
     type="revolute">
-    <limit effort="1000.0" lower="0.0" upper="6.28" velocity="0.5"/>
+    <limit lower="${-M_PI/2.0}" upper="${M_PI/2.0}" effort="50000" velocity="10000"/>
     <origin
       xyz="0.20345 -0.10209 0.11102"
-      rpy="1.2673 0.51864 1.0548" />
+      rpy="1.2673 0 1.0548" />
     <parent
       link="Chassis" />
@@ -121,7 +117,4 @@
     <axis
       xyz="0 0 -1" />
-    <limit
-      effort="0"
-      velocity="0" />
   </joint>
   <link
@@ -132,12 +125,12 @@
         rpy="0 0 0" />
       <mass
-        value="7.4055" />
+        value="7.11231" />
       <inertia
-        ixx="0.096133"
-        ixy="3.1994E-09"
-        ixz="9.2164E-10"
-        iyy="0.096133"
-        iyz="-1.1006E-09"
-        izz="0.18557" />
+        ixx="0.084989"
+        ixy="0.00"
+        ixz="0.00"
+        iyy="0.163706"
+        iyz="0.00"
+        izz="0.084989" />
     </inertial>
     <visual>
@@ -163,13 +156,23 @@
           filename="package://eklavya5_description/meshes/Front Wheel.STL" />
       </geometry>
+      <surface>
+        <friction>
+          <ode>
+            <mu>0.5</mu>
+            <mu2>0.25</mu2>
+          </ode>
+        </friction>
+        <contact>
+          <ode/>
+        </contact>
+     </surface>
     </collision>
   </link>
   <joint
     name="Steerring Wheel"
-    type="revolute">
-    <limit effort="1000.0" lower="0.0" upper="0.548" velocity="0.5"/>
+    type="continuous">
     <origin
       xyz="0.086603 0.038 0.087837"
-      rpy="1.5708 0.78607 3.1416" />
+      rpy="1.5708 0 3.1416" />
     <parent
       link="Steering" />
@@ -178,7 +181,4 @@
     <axis
       xyz="0 0 -1" />
-    <limit
-      effort="0"
-      velocity="0" />
   </joint>
   <link
@@ -189,12 +189,12 @@
         rpy="0 0 0" />
       <mass
-        value="6.735" />
+        value="6.50284" />
       <inertia
-        ixx="0.094856"
-        ixy="-4.3279E-17"
-        ixz="1.0408E-17"
-        iyy="0.18261"
-        iyz="-8.5267E-17"
-        izz="0.094856" />
+        ixx="0.084208"
+        ixy="0.00"
+        ixz="0.00"
+        iyy="0.161025"
+        iyz="0.00"
+        izz="0.084208" />
     </inertial>
     <visual>
@@ -220,10 +220,20 @@
           filename="package://eklavya5_description/meshes/Left Wheel.STL" />
       </geometry>
+      <surface>
+        <friction>
+          <ode>
+            <mu>0.5</mu>
+            <mu2>0.25</mu2>
+          </ode>
+        </friction>
+        <contact>
+          <ode/>
+        </contact>
+     </surface>
     </collision>
   </link>
   <joint
     name="LW-Chassis"
-    type="revolute">
-    <limit effort="1000.0" lower="0.0" upper="6.28" velocity="0.5"/>
+    type="continuous">
     <origin
       xyz="0.23345 -0.80043 0.41447"
@@ -235,7 +245,4 @@
     <axis
       xyz="0 -1 0" />
-    <limit
-      effort="0"
-      velocity="0" />
   </joint>
   <link
@@ -246,12 +253,12 @@
         rpy="0 0 0" />
       <mass
-        value="6.735" />
+        value="6.50284" />
       <inertia
-        ixx="0.094856"
-        ixy="-5.2042E-18"
-        ixz="-4.9061E-17"
-        iyy="0.094856"
-        iyz="1.6034E-17"
-        izz="0.18261" />
+        ixx="0.084208"
+        ixy="0.00"
+        ixz="0.00"
+        iyy="0.161025"
+        iyz="0.00"
+        izz="0.084208" />
     </inertial>
     <visual>
@@ -277,10 +284,20 @@
           filename="package://eklavya5_description/meshes/Right Wheel.STL" />
       </geometry>
+      <surface>
+        <friction>
+          <ode>
+            <mu>0.5</mu>
+            <mu2>0.25</mu2>
+          </ode>
+        </friction>
+        <contact>
+          <ode/>
+        </contact>
+     </surface>
     </collision>
   </link>
   <joint
     name="RW-Chassis"
-    type="revolute">
-    <limit effort="1000.0" lower="0.0" upper="6.28" velocity="0.5"/>
+    type="continuous">
     <origin
       xyz="0.384 -0.80043 -0.10941"
@@ -292,44 +309,205 @@
     <axis
       xyz="0 0 1" />
-    <limit
-      effort="0"
-      velocity="0" />
-  </joint>
-  <!--SENSORS-->
+  </joint>
+  <joint name="camera_joint" type="fixed">
+    <axis xyz="0 1 0" />
+    <origin xyz="0.05 0 0.5" rpy="0 0 0"/>
+    <parent link="Steering"/>
+    <child link="camera_link"/>
+  </joint>
   <!-- Camera -->
-  <sensor_camera parent="Steering" child="camera_link" name="camera" colour="Blue" camera_px="0.05" camera_py="0.0" camera_pz="0.5" camera_or="0.0" camera_op="0.0" camera_oy="0.0" axis_x="0" axis_y="1" axis_z="0"/>
-  <!-- Hokuyo Laser-->
-  <sensor_lidar parent="base_link" child="hokuyo_link" name="hokuyo" colour="Blue" lidar_px="-0.2" lidar_py="0.0" lidar_pz="0.8" lidar_or="0.0" lidar_op="0.0" lidar_oy="0.0" axis_x="0" axis_y="1" axis_z="0"/>
-  <!-- IMU-->
-  <sensor_imu parent="base_link" name="imu" colour="Blue" imu_px="-1" imu_py="0.0" imu_pz="0.8" imu_or="0.0" imu_op="0.0" imu_oy="0.0" />
-  <gazebo reference="imu_link">
-    <material>Gazebo/Blue</material>
+  <link name="camera_link">
+    <collision>
+      <origin xyz="0 0 0" rpy="0 0 0"/>
+      <geometry>
+    <box size="0.05 0.05 0.05"/>
+      </geometry>
+    </collision>
+    <visual>
+      <origin xyz="0 0 0" rpy="0 0 0"/>
+      <geometry>
+<box size="0.05 0.05 0.05"/>
+      </geometry>
+      <material name="red"/>
+    </visual>
+    <inertial>
+      <mass value="1e-5" />
+      <origin xyz="0 0 0" rpy="0 0 0"/>
+      <inertia ixx="1e-6" ixy="0" ixz="0" iyy="1e-6" iyz="0" izz="1e-6" />
+    </inertial>
+  </link>
+  <gazebo reference="camera_link">
+    <sensor type="camera" name="camera1">
+      <update_rate>24.0</update_rate>
+      <camera name="head">
+        <horizontal_fov>1.23</horizontal_fov>
+        <image>
+          <width>640</width>
+          <height>480</height>
+          <format>R8G8B8</format>
+        </image>
+        <clip>
+          <near>0.02</near>
+          <far>300</far>
+        </clip>
+        <noise>
+          <type>gaussian</type>
+          <!-- Noise is sampled independently per pixel on each frame.
+               That pixel's noise value is added to each of its color
+               channels, which at that point lie in the range [0,1]. -->
+          <mean>0.0</mean>
+          <stddev>0.007</stddev>
+        </noise>
+      </camera>
+      <plugin name="camera_controller" filename="libgazebo_ros_camera.so">
+        <alwaysOn>true</alwaysOn>
+        <updateRate>0.0</updateRate>
+        <cameraName>eklavya</cameraName>
+        <imageTopicName>image_raw</imageTopicName>
+        <cameraInfoTopicName>camera_info</cameraInfoTopicName>
+        <frameName>camera_link</frameName>
+        <hackBaseline>0.07</hackBaseline>
+        <distortionK1>0.0</distortionK1>
+        <distortionK2>0.0</distortionK2>
+        <distortionK3>0.0</distortionK3>
+        <distortionT1>0.0</distortionT1>
+        <distortionT2>0.0</distortionT2>
+      </plugin>
+    </sensor>
   </gazebo>
-    <!--${-M_PI/2.0}-->
-  <!-- GPS antenna/module -->
-  <sensor_gps parent="base_link" name="gps"
-        colour="White"
-        gps_px="-0.8"
-        gps_py="0"
-        gps_pz="0.8"
-        gps_or="0.0"
-        gps_op="0.0"
-        gps_oy="${M_PI}"
-        dimX="0.16" dimY="0.16" dimZ="0.14"/>
-  <gazebo reference="gps_link">
-      <material>Gazebo/White</material>
+<!-- Hokuyo Laser-->
+<joint name="hokuyo_joint" type="fixed">
+    <axis xyz="0 1 0" />
+    <origin xyz="-0.2 0 0.8" rpy="0 0 0"/>
+    <parent link="base_link"/>
+    <child link="hokuyo_link"/>
+  </joint>
+  <link name="hokuyo_link">
+    <collision>
+      <origin xyz="0 0 0" rpy="0 0 0"/>
+      <geometry>
+    <box size="0.025 0.025 0.025"/>
+      </geometry>
+    </collision>
+    <visual>
+      <origin xyz="0 0 0" rpy="0 0 0"/>
+      <geometry>
+        <mesh filename="package://eklavya5_description/meshes/hokuyo.dae"/>
+      </geometry>
+    </visual>
+    <inertial>
+      <mass value="1e-5" />
+      <origin xyz="0 0 0" rpy="0 0 0"/>
+      <inertia ixx="1e-6" ixy="0" ixz="0" iyy="1e-6" iyz="0" izz="1e-6" />
+    </inertial>
+  </link>
+  <!-- hokuyo -->
+  <gazebo reference="hokuyo_link">
+    <sensor type="ray" name="head_hokuyo_sensor">
+      <pose>0 0 0 0 0 0</pose>
+      <visualize>true</visualize>
+      <update_rate>40</update_rate>
+      <ray>
+        <scan>
+          <horizontal>
+            <samples>720</samples>
+            <resolution>1</resolution>
+            <min_angle>-1.570796</min_angle>
+            <max_angle>1.570796</max_angle>
+          </horizontal>
+        </scan>
+        <range>
+          <min>0.1</min>
+          <max>40.0</max>
+          <resolution>0.01</resolution>
+        </range>
+        <noise>
+          <type>gaussian</type>
+          <!-- Noise parameters based on published spec for Hokuyo laser
+               achieving "+-30mm" accuracy at range < 10m.  A mean of 0.0m and
+               stddev of 0.01m will put 99.7% of samples within 0.03m of the true
+               reading. -->
+          <mean>0.0</mean>
+          <stddev>0.01</stddev>
+        </noise>
+      </ray>
+      <plugin name="gazebo_ros_head_hokuyo_controller" filename="libgazebo_ros_laser.so">
+        <topicName>eklavya/laser/scan</topicName>
+        <frameName>hokuyo_link</frameName>
+      </plugin>
+    </sensor>
   </gazebo>
-  <!-- CONTROLS PLUGIN-->
+<!-- IMU-->
+    <sensor_imu parent="base_link" name="imu" colour="Blue" imu_px="-1" imu_py="0.0" imu_pz="0.8" imu_or="0.0" imu_op="${-M_PI/2.0}" imu_oy="0.0">
+    </sensor_imu>
+    <gazebo reference="imu_link">
+        <material>Gazebo/Blue</material>
+    </gazebo>
+    <!-- GPS antenna/module -->
+    <sensor_gps parent="base_link" name="gps"
+          colour="White"
+          gps_px="-0.8"
+          gps_py="0"
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
File: simulation/eklavya5_description/sensors/imusensor_gazebo.urdf.xacro (robot description, xacro)
@@ -12,10 +12,10 @@
         <rpyOffset>0 0 0</rpyOffset>
         <gaussianNoise>0</gaussianNoise>
-        <accelDrift>0 0 0</accelDrift>
-        <!--<accelGaussianNoise>0.35 0.35 0.3</accelGaussianNoise>-->
-        <rateDrift>0 0 0</rateDrift>
-        <!--<rateGaussianNoise>0.05 0.05 0.015</rateGaussianNoise>-->
-        <headingDrift>0</headingDrift>
-        <!--<headingGaussianNoise>0.05</headingGaussianNoise>-->
+        <accelDrift>0.5 0.5 0.5</accelDrift>
+        <accelGaussianNoise>0.35 0.35 0.3</accelGaussianNoise>
+        <rateDrift>0.1 0.1 0.1</rateDrift>
+        <rateGaussianNoise>0.05 0.05 0.015</rateGaussianNoise>
+        <headingDrift>0.1</headingDrift>
+        <headingGaussianNoise>0.05</headingGaussianNoise>
       </plugin>
     </gazebo>
